Commit message: 2025-09-29统一ros1和ros2，修改w1启动方式为xacro

File: src/robots/w1_description/urdf/w1_description.urdf (robot description, URDF)
Before this commit: robot w1_description, 23 links, 22 joints
Links:
- removed link LF_calf
- removed link LF_foot
- removed link LF_hip
- removed link LF_thigh
- removed link LF_wheel
- removed link LH_calf
- removed link LH_foot
- removed link LH_hip
- removed link LH_thigh
- removed link LH_wheel
- removed link RF_calf
- removed link RF_foot
- removed link RF_hip
- removed link RF_thigh
- removed link RF_wheel
- removed link RH_calf
- removed link RH_foot
- removed link RH_hip
- removed link RH_thigh
- removed link RH_wheel
- removed link limx_imu
- added link FL_calf, mass 1.405; collision box size=0.28 0.023 0.0451; visual mesh filename=package://w1_description/meshes/LF_calf.STL scale=1 1 1
- added link FL_foot, mass 0.995; collision cylinder length=0.017 radius=0.127; visual mesh filename=package://w1_description/meshes/LF_wheel.STL scale=1 1 1
- added link FL_hip, mass 1.543; visual mesh filename=package://w1_description/meshes/LF_hip.STL scale=1 1 1
- added link FL_thigh, mass 2.997; visual mesh filename=package://w1_description/meshes/LF_thigh.STL scale=1 1 1
- added link FR_calf, mass 1.405; collision box size=0.28 0.023 0.0451; visual mesh filename=package://w1_description/meshes/RF_calf.STL scale=1 1 1
- added link FR_foot, mass 0.995; collision cylinder length=0.017 radius=0.127; visual mesh filename=package://w1_description/meshes/RF_wheel.STL scale=1 1 1
- added link FR_hip, mass 1.543; visual mesh filename=package://w1_description/meshes/RF_hip.STL scale=1 1 1
- added link FR_thigh, mass 2.997; visual mesh filename=package://w1_description/meshes/RF_thigh.STL scale=1 1 1
- added link RL_calf, mass 1.405; collision box size=0.28 0.023 0.0451; visual mesh filename=package://w1_description/meshes/LH_calf.STL scale=1 1 1
- added link RL_foot, mass 0.995; collision cylinder length=0.017 radius=0.127; visual mesh filename=package://w1_description/meshes/LH_wheel.STL scale=1 1 1
- added link RL_hip, mass 1.543; visual mesh filename=package://w1_description/meshes/LH_hip.STL scale=1 1 1
- added link RL_thigh, mass 2.997; visual mesh filename=package://w1_description/meshes/LH_thigh.STL scale=1 1 1
- added link RR_calf, mass 1.405; collision box size=0.28 0.023 0.0451; visual mesh filename=package://w1_description/meshes/RH_calf.STL scale=1 1 1
- added link RR_foot, mass 0.995; collision cylinder length=0.017 radius=0.127; visual mesh filename=package://w1_description/meshes/RH_wheel.STL scale=1 1 1
- added link RR_hip, mass 1.543; visual mesh filename=package://w1_description/meshes/RH_hip.STL scale=1 1 1
- added link RR_thigh, mass 2.997; visual mesh filename=package://w1_description/meshes/RH_thigh.STL scale=1 1 1
- added link imu_link, mass 0.01; visual box size=0.015 0.015 0.004
Joints:
- removed joint LF_foot_fixed
- removed joint LH_foot_fixed
- removed joint RF_foot_fixed
- removed joint RH_foot_fixed
- removed joint limx_imu_joint
- added joint imu_joint: type fixed, parent trunk, child imu_link, origin xyz=0.0 0.0 0.0 rpy=0. 0. 0.
- joint FL_calf_joint: child LF_calf -> FL_calf; parent LF_thigh -> FL_thigh
- joint FL_foot_joint: child LF_wheel -> FL_foot; limit lower=-1000 upper=1000 effort=40 velocity=20 -> lower=-999999 upper=999999 effort=40 velocity=20; parent LF_calf -> FL_calf
- joint FL_hip_joint: child LF_hip -> FL_hip
- joint FL_thigh_joint: child LF_thigh -> FL_thigh; parent LF_hip -> FL_hip
- joint FR_calf_joint: child RF_calf -> FR_calf; parent RF_thigh -> FR_thigh
- joint FR_foot_joint: child RF_wheel -> FR_foot; limit lower=-1000 upper=1000 effort=40 velocity=20 -> lower=-999999 upper=999999 effort=40 velocity=20; parent RF_calf -> FR_calf
- joint FR_hip_joint: child RF_hip -> FR_hip
- joint FR_thigh_joint: child RF_thigh -> FR_thigh; parent RF_hip -> FR_hip
- joint RL_calf_joint: child LH_calf -> RL_calf; parent LH_thigh -> RL_thigh
- joint RL_foot_joint: child LH_wheel -> RL_foot; limit lower=-1000 upper=1000 effort=40 velocity=20 -> lower=-999999 upper=999999 effort=40 velocity=20; parent LH_calf -> RL_calf
- joint RL_hip_joint: child LH_hip -> RL_hip
- joint RL_thigh_joint: child LH_thigh -> RL_thigh; parent LH_hip -> RL_hip
- joint RR_calf_joint: child RH_calf -> RR_calf; parent RH_thigh -> RR_thigh
- joint RR_foot_joint: child RH_wheel -> RR_foot; limit lower=-1000 upper=1000 effort=40 velocity=20 -> lower=-999999 upper=999999 effort=40 velocity=20; parent RH_calf -> RR_calf
- joint RR_hip_joint: child RH_hip -> RR_hip
- joint RR_thigh_joint: child RH_thigh -> RR_thigh; parent RH_hip -> RR_hip
